File: debug_connector.kicad_sch (KiCad schematic)
At the start: 1 part, among them J2 Conn_ARM_JTAG_SWD_20

Commit message: Added footprint for components in Schematics. Updated LED resistors
Parts:
- J2: footprint (none) -> Connector_PinHeader_2.54mm:PinHeader_2x10_P2.54mm_Vertical
Changed lines of the file:
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@@
       (effects (font (size 1.27 1.27)) (justify right))
     )
-    (property "Footprint" "" (id 2) (at 130.175 129.54 0)
+    (property "Footprint" "Connector_PinHeader_2.54mm:PinHeader_2x10_P2.54mm_Vertical" (id 2) (at 130.175 129.54 0)
       (effects (font (size 1.27 1.27)) (justify left top) hide)
     )
