File: epaper_photo_frame.kicad_sch (KiCad schematic)
At the start: 1 part, among them J3 Battery Connector

Commit message: Added footprint for components in Schematics. Updated LED resistors
Parts:
- J3: footprint (none) -> Connector_JST:JST_PH_B2B-PH-K_1x02_P2.00mm_Vertical

Commit message: Revision 1 of the board that was manufactured
Parts:
- added H1, H2, H3, H4: MountingHole, MountingHole:MountingHole_3.2mm_M3, symbol Mechanical:MountingHole
