File: oscillator.kicad_sch (KiCad schematic)
At the start: 4 parts, among them Y1 NX3215SA-32.768K-STD-MUA-14

Commit message: Added footprint for components in Schematics. Updated LED resistors
Parts:
- C31, C32: footprint (none) -> Capacitor_SMD:C_0402_1005Metric
- R7: footprint (none) -> Resistor_SMD:R_0402_1005Metric
Changed lines of the file:
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@@
       (effects (font (size 1.27 1.27)) (justify left))
     )
-    (property "Footprint" "" (id 2) (at 155.575 87.63 0)
+    (property "Footprint" "Capacitor_SMD:C_0402_1005Metric" (id 2) (at 155.575 87.63 0)
       (effects (font (size 1.27 1.27)) hide)
     )
@@
       (effects (font (size 1.27 1.27)) (justify left))
     )
-    (property "Footprint" "" (id 2) (at 129.54 87.63 0)
+    (property "Footprint" "Capacitor_SMD:C_0402_1005Metric" (id 2) (at 129.54 87.63 0)
       (effects (font (size 1.27 1.27)) hide)
     )
@@
       (effects (font (size 1.27 1.27)) (justify left))
     )
-    (property "Footprint" "" (id 2) (at 162.56 62.865 0)
+    (property "Footprint" "Resistor_SMD:R_0402_1005Metric" (id 2) (at 162.56 62.865 0)
       (effects (font (size 1.27 1.27)) hide)
     )

Commit message: Revision 1 of the board that was manufactured
Parts:
- C31, C32: LCSC (none) -> C730435
- R7: LCSC (none) -> C17168
- Y1: LCSC (none) -> C156244
