File: display_adapter.kicad_sch (KiCad schematic)
At the start: 60 parts, among them J4 54104-5031, Q1 BSS138, Q2 SI2301CDS-T1-E3, Q31 AO3401A, Q32 S8050, U2 RT9193-33GB

Commit message: Added footprint for components in Schematics. Updated LED resistors
Parts:
- C1, C10, C11, C12, C18, C19, C2, C20, C21, C23, C24, C25, C26, C27, C28, C29, C3, C4, C5, C6, C7, C8, C9: footprint (none) -> Capacitor_SMD:C_0201_0603Metric
- C14, C15, C16, C17: footprint (none) -> Capacitor_SMD:C_0805_2012Metric
- L1, L2: footprint (none) -> SamacSys_Parts:INDPM4040X200N
- NT1, NT2, NT3, NT4, NT5, NT6, NT7, NT8: footprint (none) -> NetTie:NetTie-2_SMD_Pad2.0mm
- Q32: footprint Package_TO_SOT_THT:TO-92_Inline -> Package_TO_SOT_SMD:SOT-23
- R1, R2, R27, R3, R33, R34, R35, R36, R37, R4, R5, RA1, RB1: footprint (none) -> Resistor_SMD:R_0805_2012Metric

Commit message: Added preliminary PCL layout
Parts:
- C1, C10, C11, C12, C18, C19, C2, C20, C21, C23, C24, C25, C26, C27, C28, C29, C3, C4, C5, C6, C7, C8, C9: footprint Capacitor_SMD:C_0201_0603Metric -> Capacitor_SMD:C_0603_1608Metric
- NT1, NT2, NT3, NT4, NT5, NT6, NT7, NT8: footprint NetTie:NetTie-2_SMD_Pad2.0mm -> NetTie:NetTie-2_SMD_Pad0.5mm
Connections:
- net EPD_D1: no longer names the net of J4.34
- net EPD_D2: no longer names the net of J4.35
- net EPD_D3: no longer names the net of J4.36
- no-connect marks 8 -> 11

Commit message: Revision 1 of the board that was manufactured
Parts:
- C1: LCSC (none) -> C19666; MAX Voltage (none) -> 10V; MAX voltage 10V -> (none)
- C10, C12, C21, C28, C3, C5, C6, C7, C8, C9: LCSC (none) -> C96446
- C11, C18, C24, C25, C26, C29: LCSC (none) -> C15849
- C14, C15: LCSC (none) -> C49678
- C16: LCSC (none) -> C28323
- C17: LCSC (none) -> C1729
- C19, C20: LCSC (none) -> C19666
- C2, C27: LCSC (none) -> C1623
- C23: LCSC (none) -> C23630
- C4: LCSC (none) -> C14663
- D1, D2, D3, D4: LCSC (none) -> C18863
- J4: LCSC (none) -> C505282
- L1, L2: LCSC (none) -> C82398
- Q1: LCSC (none) -> C82045
- Q2: LCSC (none) -> C145226
- Q31: LCSC (none) -> C15127
- Q32: footprint Package_TO_SOT_SMD:SOT-23 -> Package_TO_SOT_SMD:SOT-23-3; LCSC (none) -> C2150
- R1, R4: LCSC (none) -> C441966
- R2, R5: LCSC (none) -> C491238
- R27: LCSC (none) -> C149504
- R3, RA1, RB1: LCSC (none) -> C17477
- R33, R34: LCSC (none) -> C17713
- R35: LCSC (none) -> C510098
- R36: LCSC (none) -> C17513
- R37: LCSC (none) -> C2073899
- U2: LCSC (none) -> C15651

Commit message: Fix NPN BJT Base and emitter pin swap. Attach BS0 to GND to select 4 pin SPI mode for Epaper display. Use 2 side FPC connector
Parts:
- removed J4: 54104-5031, SamacSys_Parts:541045031, symbol SamacSys_Parts:54104-5031
- removed Q32: S8050, Package_TO_SOT_SMD:SOT-23-3, symbol Transistor_BJT:S8050
- added J4: XF2M50151A, SamacSys_Parts:XF2M50151A, symbol SamacSys_Parts:XF2M50151A
- added Q32: MMSS8050, Package_TO_SOT_SMD:SOT-23, symbol PCM_Transistor_BJT_AKL:MMSS8050
- R37: LCSC C2073899 -> C17713
Connections:
- net 3v3: no longer NT4.2
- net BS0: now also J4.26
- net BS1: now also J4.27
- net CP1N: now also J4.45
- net CP1P: now also J4.46
- net CP2N: now also J4.42
- net CP2P: now also J4.43
- net EPD_BUSY: now also J4.29
- net EPD_CS: now also J4.31
- net EPD_DC: now also J4.30
- net EPD_DIN: now also J4.33
- net EPD_RST: now also J4.28
- net EPD_RST_INT: now also Q32.1 (B)
- net EPD_SCK: now also J4.32
- net FPL VCOM: now also J4.3
- net GDRC: now also J4.9
- net GDRH: now also J4.5
- net GND: now also NT4.2, Q32.2 (E)
- net GNDA+(GND): now also J4.12, J4.21
- net GNDA/GND: now also J4.39
- net REFN: now also J4.22
- net REFP: now also J4.23
- net RESEC: now also J4.10
- net RESEH: now also J4.6
- net RESEL: now also J4.8
- net TFT VCOM: now also J4.2
- net VCC_DIS_PU: now also Q32.3 (C)
- net VCOMBD: now also J4.50
- net VCP1: now also J4.44
- net VCP2: now also J4.41
- net VDD: now also J4.38, J4.4
- net VDDD/VDDDO: now also J4.37
- net VDDIO: now also J4.40
- net VGH: now also J4.49
- net VGL: now also J4.13
- net VPC: now also J4.11
- net VPH: now also J4.14
- net VSH: now also J4.15
- net VSH LV: now also J4.16
- net VSH LV2: now also J4.17
- net VSL: now also J4.18
- net VSL LV: now also J4.19
- net VSL LV2: now also J4.20
Other:
- note added: "BS0 pulled low to chose 4-line SPI"
- note removed: "BS0 pulled high to chose 3-line SPI"
- moved on the sheet: NT4
